Commit message: add spresense imu

File: orange_description/xacro/orange_robot.xacro (robot description, xacro)
@@ -12,5 +12,5 @@
   <xacro:include filename="$(find orange_description)/xacro/sensors/livox.xacro"/>
   <xacro:sensor_livox name="livox_frame" parent="base_link" min_angle="-2.35619" max_angle="2.35619" samples="720">
-    <origin xyz="-0.0185 0.0 0.8985" rpy="${pi} 0.0 0.0"/>
+    <origin xyz="-0.0185 0.0 0.94" rpy="${pi} 0.0 0.0"/>
   </xacro:sensor_livox>
   <!--simulation-->

Commit message: add lidar 2 description in xacro file

File: orange_description/xacro/orange_robot.xacro (robot description, xacro)
@@ -13,4 +13,7 @@
   <xacro:sensor_livox name="livox_frame" parent="base_link" min_angle="-2.35619" max_angle="2.35619" samples="720">
     <origin xyz="-0.0185 0.0 0.94" rpy="${pi} 0.0 0.0"/>
+  </xacro:sensor_livox>
+  <xacro:sensor_livox name="livox_under" parent="base_link" min_angle="-2.35619" max_angle="2.35619" samples="720">
+    <origin xyz="-0.0185 0.0 0.67" rpy="${pi} 0.0 0.0"/>
   </xacro:sensor_livox>
   <!--simulation-->
